File: pcb_epsilon/Epsilon/Epsilon.kicad_pcb (KiCad board)
At the start: 2 copper layers, 69 x 31.5 mm, 18 parts, among them J1 SG1m, J2 SG2p, J3 SG1p, J4 SG2m, Q1 AO3401A, U1 ADA4940-1ARZ-R7, U2 DS28E07P+T

Commit message: Updated Epsilon PCB and Ozys Sch
Parts:
- J1, J2, J3, J4: footprint Connector_Wire:SolderWirePad_1x01_SMD_5x10mm -> Connector_Wire:SolderWirePad_1x01_SMD_1x2mm
- R1, R2, R3, R4: footprint Resistor_SMD:R_0402_1005Metric_Pad0.72x0.64mm_HandSolder -> Resistor_SMD:R_0603_1608Metric_Pad0.98x0.95mm_HandSolder
- R6, R7: footprint Resistor_SMD:R_0805_2012Metric_Pad1.20x1.40mm_HandSolder -> Resistor_SMD:R_0402_1005Metric_Pad0.72x0.64mm_HandSolder
