File: epsilon/Epsilon_final/Epsilon_final.kicad_sch (KiCad schematic)
At the start: 16 parts, among them J3 Conn_01x02_Pin, J4 Conn_01x02_Pin, Q5 AO3401A, U12 ADA4940-1ARZ-R7, U8 DS28E07P+T

Commit message: Yolo2
new Ozys
Parts:
- removed Audio2: PJ-3200B-4A, Rocketry_Easyeda:AUDIO-TH_PJ-3200B-4A, symbol Rocketry_Easyeda:PJ-3200B-4A
- removed C29, C30: 100n, Capacitor_SMD:C_0402_1005Metric, symbol Device:C
- removed C31: 1000p, Capacitor_SMD:C_0402_1005Metric, symbol Device:C
- removed J3, J4: Conn_01x02_Pin, symbol Connector:Conn_01x02_Pin
- removed Q5: AO3401A, Package_TO_SOT_SMD:SOT-23, symbol Transistor_FET:AO3401A
- removed R20: 10K, symbol Device:R
- removed R21, R22: 330R, Resistor_SMD:R_0805_2012Metric_Pad1.20x1.40mm_HandSolder, symbol Device:R
- removed R46, R48: 510K, symbol Device:R
- removed R47, R49: 5.6K, symbol Device:R
- removed U12: ADA4940-1ARZ-R7, Rocketry_Easyeda:SOIC-8_L4.9-W3.9-P1.27-LS6.0-BL, symbol Rocketry_Easyeda:ADA4940-1ARZ-R7
- removed U8: DS28E07P+T, Rocketry_Easyeda:TSOC-6_L3.9-W4.3-P1.27-BL, symbol Rocketry_Easyeda:DS28E07P+T
- added Audio1: PJ-3200B-4A, Rocketry_Easyeda:AUDIO-TH_PJ-3200B-4A, symbol Rocketry_Easyeda:PJ-3200B-4A
- added C1, C3: 100n, Capacitor_SMD:C_0402_1005Metric, symbol Device:C
- added C2: 1000p, Capacitor_SMD:C_0402_1005Metric, symbol Device:C
- added J1: SG1p, Connector_Wire:SolderWirePad_1x01_SMD_1x2mm, symbol Connector:Conn_01x01_Pin
- added J2: SG1m, Connector_Wire:SolderWirePad_1x01_SMD_1x2mm, symbol Connector:Conn_01x01_Pin
- added J3: SG2p, Connector_Wire:SolderWirePad_1x01_SMD_1x2mm, symbol Connector:Conn_01x01_Pin
- added J4: SG2m, Connector_Wire:SolderWirePad_1x01_SMD_1x2mm, symbol Connector:Conn_01x01_Pin
- added Q1: AO3401A, Package_TO_SOT_SMD:SOT-23, symbol Transistor_FET:AO3401A
- added R1, R2: 330K, Resistor_SMD:R_0603_1608Metric_Pad0.98x0.95mm_HandSolder, symbol Device:R
- added R3, R4: 6.8K, Resistor_SMD:R_0603_1608Metric_Pad0.98x0.95mm_HandSolder, symbol Device:R
- added R5: 10K, Resistor_SMD:R_0402_1005Metric_Pad0.72x0.64mm_HandSolder, symbol Device:R
- added U1: ADA4940-1ARZ-R7, Rocketry_Easyeda:SOIC-8_L4.9-W3.9-P1.27-LS6.0-BL, symbol Rocketry_Easyeda:ADA4940-1ARZ-R7
- added U2: DS28E07P+T, Rocketry_Easyeda:TSOC-6_L3.9-W4.3-P1.27-BL, symbol Rocketry_Easyeda:DS28E07P+T
Connections:
- net 3V3A_SW: now also Audio1.3, C1.1, C2.2, J1.1 (Pin_1), Q1.2 (S), R5.1, U1.3 (+VS)
- net GND: now also Audio1.1, C1.2, C2.1, C3.1, J4.1 (Pin_1), Q1.3 (D), U1.6 (–VS), U2.1 (GND)
- new net: R1.2, R3.1, U1.8 (+IN)
- new net: J2.1 (Pin_1), R3.2
- new net: Q1.1 (G), R5.2, U2.2 (IO)
- new net: C3.2, U1.2 (VOCM)
- new net: R2.2, R4.1, U1.1 (–IN)
- new net: J3.1 (Pin_1), R4.2
- new net: Audio1.4, R2.1, U1.4 (+OUT)
- new net: Audio1.2, R1.1, U1.5 (–OUT)

Commit message: OZYS and EPSILON schematics updated.
OZYS
- New 3.5 PJ-320A-4P DIP
- Fixed TPS Regulator Connections
- Fixed STM32 Connections
- Added Associated .ioc for stm32 pin config
- Loading Capacitance of LSE based off  an5093 STM datasheet
EPSILON
- same 3.5 as OZYS
Parts:
- removed Audio1: PJ-3200B-4A, Rocketry_Easyeda:AUDIO-TH_PJ-3200B-4A, symbol Rocketry_Easyeda:PJ-3200B-4A
- added J5: AudioJack4, Rocketry_Easyeda:AUDIO-TH_PJ-320A-4P-DIP, symbol Connector_Audio:AudioJack4
Connections:
- net 3V3A_SW: now also J5.R2
- net GND: now also J5.S
- net at R2.1, U1.4 (+OUT): now also J5.T
- net at R1.1, U1.5 (–OUT): now also J5.R1
Changed lines of the file:
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@@
-	(wire
-		(pts
-			(xy 82.55 97.79) (xy 78.74 97.79)
-		)
-		(stroke
-			(width 0)
-			(type default)
-		)
-	)
 	(wire
 		(pts
@@
 	(wire
 		(pts
+			(xy 73.66 102.87) (xy 115.57 102.87)
+		)
+		(stroke
+			(width 0)
+			(type default)
+		)
+	)
+	(wire
+		(pts
 			(xy 201.93 114.3) (xy 179.07 114.3)
 		)
@@
 	(wire
 		(pts
+			(xy 115.57 102.87) (xy 115.57 114.3)
+		)
+		(stroke
+			(width 0)
+			(type default)
+		)
+	)
+	(wire
+		(pts
 			(xy 201.93 114.3) (xy 201.93 105.41)
 		)
@@
 	(wire
 		(pts
-			(xy 109.22 95.25) (xy 78.74 95.25)
-		)
-		(stroke
-			(width 0)
-			(type default)
-		)
-	)
-	(wire
-		(pts
 			(xy 217.17 113.03) (xy 217.17 124.46)
 		)
@@
 	(wire
 		(pts
-			(xy 109.22 114.3) (xy 115.57 114.3)
-		)
-		(stroke
-			(width 0)
-			(type default)
-		)
-	)
-	(wire
-		(pts
-			(xy 87.63 105.41) (xy 87.63 102.87)
-		)
-		(stroke
-			(width 0)
-			(type default)
-		)
-	)
-	(wire
-		(pts
 			(xy 201.93 97.79) (xy 233.68 97.79)
 		)
@@
 	(wire
 		(pts
-			(xy 82.55 86.36) (xy 132.08 86.36)
+			(xy 115.57 86.36) (xy 132.08 86.36)
 		)
 		(stroke
@@
 	(wire
 		(pts
+			(xy 115.57 100.33) (xy 73.66 100.33)
+		)
+		(stroke
+			(width 0)
+			(type default)
+		)
+	)
+	(wire
+		(pts
 			(xy 158.75 114.3) (xy 158.75 139.7)
 		)
@@
 	(wire
 		(pts
-			(xy 109.22 95.25) (xy 109.22 114.3)
-		)
-		(stroke
-			(width 0)
-			(type default)
-		)
-	)
-	(wire
-		(pts
 			(xy 130.81 120.65) (xy 143.51 120.65)
 		)
@@
 	(wire
 		(pts
+			(xy 73.66 95.25) (xy 80.01 95.25)
+		)
+		(stroke
+			(width 0)
+			(type default)
+		)
+	)
+	(wire
+		(pts
 			(xy 162.56 44.45) (xy 171.45 44.45)
 		)
@@
 	(wire
 		(pts
-			(xy 78.74 102.87) (xy 87.63 102.87)
+			(xy 73.66 97.79) (xy 78.74 97.79)
 		)
 		(stroke
@@
 	(wire
 		(pts
-			(xy 82.55 86.36) (xy 82.55 97.79)
-		)
-		(stroke
-			(width 0)
-			(type default)
-		)
-	)
-	(wire
-		(pts
 			(xy 115.57 139.7) (xy 139.7 139.7)
 		)
@@
 	(wire
 		(pts
-			(xy 92.71 105.41) (xy 87.63 105.41)
+			(xy 115.57 86.36) (xy 115.57 100.33)
 		)
 		(stroke
@@
 		(pts
 			(xy 148.59 86.36) (xy 158.75 86.36)
-		)
-		(stroke
-			(width 0)
-			(type default)
-		)
-	)
-	(wire
-		(pts
-			(xy 78.74 100.33) (xy 92.71 100.33)
 		)
 		(stroke
@@
 	)
 	(symbol
+		(lib_id "Connector_Audio:AudioJack4")
+		(at 68.58 97.79 0)
+		(unit 1)
+		(exclude_from_sim no)
+		(in_bom yes)
+		(on_board yes)
+		(dnp no)
+		(fields_autoplaced yes)
+		(property "Reference" "J5"
+			(at 66.04 88.9 0)
+			(effects
+				(font
+					(size 1.27 1.27)
+				)
+			)
+		)
+		(property "Value" "AudioJack4"
+			(at 66.04 91.44 0)
+			(effects
+				(font
+					(size 1.27 1.27)
+				)
+			)
+		)
+		(property "Footprint" "Rocketry_Easyeda:AUDIO-TH_PJ-320A-4P-DIP"
+			(at 68.58 97.79 0)
+			(effects
+				(font
+					(size 1.27 1.27)
+				)
+				(hide yes)
+			)
+		)
+		(property "Datasheet" "~"
+			(at 68.58 97.79 0)
+			(effects
+				(font
+					(size 1.27 1.27)
+				)
+				(hide yes)
+			)
+		)
+		(property "Description" "Audio Jack, 4 Poles (TRRS)"
+			(at 68.58 97.79 0)
+			(effects
+				(font
+					(size 1.27 1.27)
+				)
+				(hide yes)
+			)
+		)
+		(pin "S"
+		)
+		(pin "R2"
+		)
+		(pin "R1"
+		)
+		(pin "T"
+		)
+		(instances
+			(project ""
+				(path "/b0321cc8-d802-43c8-a38f-bba100abf2a4"
+					(reference "J5")
+					(unit 1)
+				)
+			)
+		)
+	)
+	(symbol
 		(lib_id "power:GND")
 		(at 123.19 125.73 270)
@@
 	(symbol
 		(lib_id "power:+3.3V")
-		(at 92.71 100.33 270)
+		(at 78.74 97.79 270)
 		(mirror x)
 		(unit 1)
@@
 		(fields_autoplaced yes)
 		(property "Reference" "#PWR01"
-			(at 88.9 100.33 0)
+			(at 74.93 97.79 0)
 			(effects
 				(font
@@
 		)
 		(property "Value" "3V3A_SW"
-			(at 96.52 100.3299 90)
+			(at 82.55 97.7899 90)
 			(effects
 				(font
@@
 		)
 		(property "Footprint" ""
-			(at 92.71 100.33 0)
+			(at 78.74 97.79 0)
 			(effects
 				(font
@@
 		)
 		(property "Datasheet" ""
-			(at 92.71 100.33 0)
+			(at 78.74 97.79 0)
 			(effects
 				(font
@@
 		)
 		(property "Description" "Power symbol creates a global label with name \"+3.3V\""
-			(at 92.71 100.33 0)
+			(at 78.74 97.79 0)
 			(effects
 				(font
@@
 	)
 	(symbol
-		(lib_id "Rocketry_Easyeda:PJ-3200B-4A")
-		(at 69.85 100.33 0)
-		(mirror x)
-		(unit 1)
-		(exclude_from_sim no)
-		(in_bom yes)
-		(on_board yes)
-		(dnp no)
-		(property "Reference" "Audio1"
-			(at 59.69 100.3301 0)
-			(effects
-				(font
-					(size 1.27 1.27)
-				)
-				(justify right)
-			)
-		)
-		(property "Value" "PJ-3200B-4A"
-			(at 59.69 97.7901 0)
-			(effects
-				(font
-					(size 1.27 1.27)
-				)
-				(justify right)
-			)
-		)
-		(property "Footprint" "Rocketry_Easyeda:AUDIO-TH_PJ-3200B-4A"
-			(at 69.85 87.63 0)
-			(effects
-				(font
-					(size 1.27 1.27)
-				)
-				(hide yes)
-			)
-		)
-		(property "Datasheet" "https://lcsc.com/product-detail/Audio-Connectors_PJ-3200B-4A_C136687.html"
-			(at 69.85 85.09 0)
-			(effects
-				(font
-					(size 1.27 1.27)
-				)
-				(hide yes)
-			)
-		)
-		(property "Description" ""
-			(at 69.85 100.33 0)
-			(effects
-				(font
-					(size 1.27 1.27)
-				)
-				(hide yes)
-			)
-		)
-		(property "LCSC Part" "C136687"
-			(at 69.85 82.55 0)
-			(effects
-				(font
-					(size 1.27 1.27)
-				)
-				(hide yes)
-			)
-		)
-		(pin "3"
-		)
-		(pin "4"
-		)
-		(pin "1"
-		)
-		(pin "2"
-		)
-		(instances
-			(project "Epsilon_final"
-				(path "/b0321cc8-d802-43c8-a38f-bba100abf2a4"
-					(reference "Audio1")
-					(unit 1)
-				)
-			)
-		)
-	)
-	(symbol
 		(lib_id "Rocketry_Easyeda:ADA4940-1ARZ-R7")
 		(at 146.05 99.06 270)
@@
 	(symbol
 		(lib_id "power:GND")
-		(at 92.71 105.41 90)
+		(at 80.01 95.25 90)
 		(unit 1)
 		(exclude_from_sim no)
@@
 		(dnp no)
 		(property "Reference" "#PWR02"
-			(at 99.06 105.41 0)
+			(at 86.36 95.25 0)
 			(effects
 				(font
@@
 		)
 		(property "Value" "GND"
-			(at 97.79 105.41 90)
+			(at 85.09 95.25 90)
 			(effects
 				(font
@@
 		)
 		(property "Footprint" ""
-			(at 92.71 105.41 0)
+			(at 80.01 95.25 0)
 			(effects
 				(font
@@
 		)
 		(property "Datasheet" ""
-			(at 92.71 105.41 0)
+			(at 80.01 95.25 0)
 			(effects
 				(font
@@
 		)
 		(property "Description" "Power symbol creates a global label with name \"GND\" , ground"
-			(at 92.71 105.41 0)
-			(effects
-				(font
+			(at 80.01 95.25 0)
+			(effects
+				(font
