File: ozyz_v3/Power.kicad_sch (KiCad schematic)
At the start: 26 parts, among them J2 Conn_01x02_Pin, Q1 AO3401A, Q2 AO3401A, U4 TPS63070RNMR

Commit message: OZYS ready for layout
Parts:
- removed D1: SS34, Diode_SMD:D_SMA, symbol Diode:SS34
- removed L1, L3: SPM6530T-1R5M100, Rocketry_Easyeda:IND-SMD_L7.1-W6.5-P5.60, symbol Rocketry_Easyeda:SPM6530T-1R5M100
- removed Q1: AO3401A, Package_TO_SOT_SMD:SOT-23, symbol Transistor_FET:AO3401A
- removed R13: 150k, Resistor_SMD:R_0603_1608Metric, symbol Device:R
- added C43, C44: 22u, Capacitor_SMD:C_0603_1608Metric, symbol Device:C
- added D2: 1N5819WS, Diode_SMD:D_SOD-323, symbol Diode:1N5819WS
- added Q1: AO3400A, Rocketry_Easyeda:SOT-23-3_L2.9-W1.3-P1.90-LS2.4-BR, symbol Rocketry_Easyeda:AO3400A
- added U10, U11: FTC252012S1R5MBCA (1.5uF 2.9A), Rocketry_Easyeda:IND-SMD_L2.5-W2.0_MEKK2520TR47M, symbol Rocketry_Easyeda:FTC252012S1R5MBCA (1.5uF 2.9A)
- R11, R7: footprint Resistor_SMD:R_0603_1608Metric -> Resistor_SMD:R_0402_1005Metric
Connections:
- net +3V3A: now also C43.2, C44.2, U10.2
- net 3V3A_SW: now also Q1.3 (D)
- net 3V3A_SW_EN: now also Q1.1 (G)
- net GND: now also C43.1, C44.1, Q1.2 (S)
- net VBUS: now also D2.2 (A)
- net at C14.2, C15.2, C16.2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: now also J2.1 (Pin_1), R8.2, D2.1 (K)
- net at U4.11 (L1): now also U11.1
- net at U4.9 (L2): now also U11.2
- net +3.3V renamed +3V3
- net +3V3: now also U10.1
Other:
- moved on the sheet: Q2
