File: ozyz_v3/Receiver1.kicad_sch (KiCad schematic)
At the start: 14 parts, among them J5 AudioJack4, Q7 AO3401A, Q8 2N7002

Commit message: epsilon ready for layout
Parts:
- removed Q7: AO3401A, Package_TO_SOT_SMD:SOT-23, symbol Transistor_FET:AO3401A
- removed R25: 10K, symbol Device:R

Commit message: OZYS ready for layout
Parts:
- removed C22, C28: 500nF, symbol Device:C
- removed R30: 33K, Resistor_SMD:R_0402_1005Metric, symbol Device:R
- added C2, C7: 1nF 1%, Capacitor_SMD:C_0603_1608Metric_Pad1.08x0.95mm_HandSolder, symbol Device:C
- added R13, R14: 2.4k 1%, Capacitor_SMD:C_0603_1608Metric_Pad1.08x0.95mm_HandSolder, symbol Device:R
- C32, C36: value 500nF -> 1nF 1%; footprint (none) -> Capacitor_SMD:C_0603_1608Metric_Pad1.08x0.95mm_HandSolder
- J5: footprint Rocketry_Easyeda:AUDIO-TH_PJ-320A-4P-DIP -> Rocketry_Manual:AUDIO-TH_PJ-320A-4P-DIP
- R22, R34: value 15 -> 2.4k 1%; footprint (none) -> Capacitor_SMD:C_0603_1608Metric_Pad1.08x0.95mm_HandSolder
- R27: value 15 -> 51R; footprint (none) -> Resistor_SMD:R_0402_1005Metric
Connections:
- net DIFFERENTIAL_M: now also C2.1, R13.1; no longer C32.1, R34.1
- net DIFFERENTIAL_P: now also C7.2, R14.1; no longer C36.2, R22.1
- net GND: now also C2.2, C7.1
- net ONE_WIRE_OUT: now reaches J5.R2, R27.2
- net +3.3V renamed +3V3
- new net: C36.2, R14.2, R22.1
- new net: C32.1, R13.2, R34.1
Other:
- moved on the sheet: C32, C36, J5, LED3, Q8, R22, R26, R27, R34

Commit message: update connector placement
Parts:
- renumbered C2 to C26, C7 to C27, R13 to R25, R14 to R30
Changed lines of the file:
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@@
 		(on_board yes)
 		(dnp no)
-		(property "Reference" "#PWR080"
+		(property "Reference" "#PWR082"
 			(at 173.99 93.98 0)
 			(effects
@@
 		(dnp no)
 		(fields_autoplaced yes)
-		(property "Reference" "C2"
+		(property "Reference" "C26"
 			(at 167.64 87.6299 0)
 			(effects
@@
 		(dnp no)
 		(fields_autoplaced yes)
-		(property "Reference" "R13"
+		(property "Reference" "R25"
 			(at 156.21 76.2 90)
 			(effects
@@
 		(dnp no)
 		(fields_autoplaced yes)
-		(property "Reference" "R14"
+		(property "Reference" "R30"
 			(at 156.21 99.06 90)
 			(effects
@@
 		(dnp no)
 		(fields_autoplaced yes)
-		(property "Reference" "C7"
+		(property "Reference" "C27"
 			(at 167.64 97.7899 0)
 			(effects
@@
 		(on_board yes)
 		(dnp no)
-		(property "Reference" "#PWR049"
+		(property "Reference" "#PWR054"
 			(at 127 142.24 0)
 			(effects

Commit message: Got rid of LED Fet
- restructuring
Parts:
- removed Q8: 2N7002, Rocketry_Easyeda:SOT-23-3_L2.9-W1.3-P1.90-LS2.4-BR, symbol Rocketry_Easyeda:2N7002
- removed R26: 33R, Resistor_SMD:R_0402_1005Metric, symbol Device:R
- added R15: 220R, Resistor_SMD:R_0402_1005Metric, symbol Device:R
Connections:
- net GND: now also R15.2
- net LED_SW: now also LED3.1 (A)
- net at LED3.2 (K): now also R15.1
Changed lines of the file:
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@@
-	(wire
-		(pts
-			(xy 172.72 142.24) (xy 184.15 142.24)
-		)
-		(stroke
-			(width 0)
-			(type default)
-		)
-	)
 	(wire
 		(pts
@@
 	(wire
 		(pts
+			(xy 171.45 142.24) (xy 184.15 142.24)
+		)
+		(stroke
+			(width 0)
+			(type default)
+		)
+	)
+	(wire
+		(pts
 			(xy 134.62 105.41) (xy 138.43 105.41)
 		)
@@
 	(wire
 		(pts
-			(xy 123.19 142.24) (xy 127 142.24)
-		)
-		(stroke
-			(width 0)
-			(type default)
-		)
-	)
-	(wire
-		(pts
 			(xy 134.62 142.24) (xy 140.97 142.24)
 		)
@@
 	(wire
 		(pts
-			(xy 167.64 154.94) (xy 167.64 149.86)
-		)
-		(stroke
-			(width 0)
-			(type default)
-		)
-	)
-	(wire
-		(pts
 			(xy 134.62 82.55) (xy 138.43 82.55)
 		)
@@
 	(wire
 		(pts
-			(xy 163.83 154.94) (xy 167.64 154.94)
-		)
-		(stroke
-			(width 0)
-			(type default)
-		)
-	)
-	(wire
-		(pts
 			(xy 127 105.41) (xy 120.65 105.41)
 		)
@@
 	(wire
 		(pts
-			(xy 151.13 142.24) (xy 162.56 142.24)
+			(xy 151.13 142.24) (xy 163.83 142.24)
 		)
 		(stroke
@@
 	(hierarchical_label "LED_SW"
 		(shape input)
-		(at 163.83 154.94 180)
+		(at 134.62 142.24 180)
 		(effects
 			(font
@@
 	)
 	(symbol
-		(lib_id "Rocketry_Easyeda:2N7002")
-		(at 167.64 144.78 90)
+		(lib_id "Device:R")
+		(at 167.64 142.24 90)
 		(unit 1)
 		(exclude_from_sim no)
@@
 		(dnp no)
 		(fields_autoplaced yes)
-		(property "Reference" "Q8"
-			(at 167.64 133.35 90)
-			(effects
-				(font
-					(size 1.27 1.27)
-				)
-			)
-		)
-		(property "Value" "2N7002"
+		(property "Reference" "R15"
 			(at 167.64 135.89 90)
 			(effects
@@
 			)
 		)
-		(property "Footprint" "Rocketry_Easyeda:SOT-23-3_L2.9-W1.3-P1.90-LS2.4-BR"
-			(at 180.34 144.78 0)
-			(effects
-				(font
-					(size 1.27 1.27)
-				)
-				(hide yes)
-			)
-		)
-		(property "Datasheet" "https://lcsc.com/product-detail/MOSFET_2N7002-7002_C8545.html"
-			(at 182.88 144.78 0)
-			(effects
-				(font
-					(size 1.27 1.27)
-				)
-				(hide yes)
-			)
-		)
-		(property "Description" ""
-			(at 167.64 144.78 0)
-			(effects
-				(font
-					(size 1.27 1.27)
-				)
-				(hide yes)
-			)
-		)
-		(property "LCSC Part" "C8545"
-			(at 185.42 144.78 0)
+		(property "Value" "220R"
+			(at 167.64 138.43 90)
+			(effects
+				(font
+					(size 1.27 1.27)
+				)
+			)
+		)
+		(property "Footprint" "Resistor_SMD:R_0402_1005Metric"
+			(at 167.64 144.018 90)
+			(effects
+				(font
+					(size 1.27 1.27)
+				)
+				(hide yes)
+			)
+		)
+		(property "Datasheet" "~"
+			(at 167.64 142.24 0)
+			(effects
+				(font
+					(size 1.27 1.27)
+				)
+				(hide yes)
+			)
+		)
+		(property "Description" "Resistor"
+			(at 167.64 142.24 0)
 			(effects
 				(font
@@
 		)
 		(pin "2"
-		)
-		(pin "3"
 		)
 		(instances
 			(project "OZYS_V3_Final"
 				(path "/2ecddb92-e766-42eb-adbc-b6d17a65e8ea/55853f5b-0992-495b-b96a-8743589b5403"
-					(reference "Q8")
+					(reference "R26")
 					(unit 1)
 				)
 				(path "/2ecddb92-e766-42eb-adbc-b6d17a65e8ea/6e4545c6-9e5c-4e6b-94f2-451b2f16f4ae"
-					(reference "Q4")
+					(reference "R17")
 					(unit 1)
 				)
 				(path "/2ecddb92-e766-42eb-adbc-b6d17a65e8ea/92ea14e4-7796-41b2-9af7-4cb5ffd88b52"
-					(reference "Q6")
+					(reference "R15")
 					(unit 1)
 				)
 				(path "/2ecddb92-e766-42eb-adbc-b6d17a65e8ea/d66c3d32-3008-485f-b8d3-7e1a6a0b22a4"
-					(reference "Q10")
+					(reference "R32")
 					(unit 1)
 				)
@@
 	(symbol
 		(lib_id "Device:R")
-		(at 130.81 142.24 90)
-		(unit 1)
-		(exclude_from_sim no)
-		(in_bom yes)
-		(on_board yes)
-		(dnp no)
-		(fields_autoplaced yes)
-		(property "Reference" "R26"
-			(at 130.81 135.89 90)
-			(effects
-				(font
-					(size 1.27 1.27)
-				)
-			)
-		)
-		(property "Value" "33R"
-			(at 130.81 138.43 90)
-			(effects
-				(font
-					(size 1.27 1.27)
-				)
-			)
-		)
-		(property "Footprint" "Resistor_SMD:R_0402_1005Metric"
-			(at 130.81 144.018 90)
-			(effects
-				(font
-					(size 1.27 1.27)
-				)
-				(hide yes)
-			)
-		)
-		(property "Datasheet" "~"
-			(at 130.81 142.24 0)
-			(effects
-				(font
-					(size 1.27 1.27)
-				)
-				(hide yes)
-			)
-		)
-		(property "Description" "Resistor"
-			(at 130.81 142.24 0)
-			(effects
-				(font
-					(size 1.27 1.27)
-				)
-				(hide yes)
-			)
-		)
-		(pin "1"
-		)
-		(pin "2"
-		)
-		(instances
-			(project "OZYS_V3_Final"
-				(path "/2ecddb92-e766-42eb-adbc-b6d17a65e8ea/55853f5b-0992-495b-b96a-8743589b5403"
-					(reference "R26")
-					(unit 1)
-				)
-				(path "/2ecddb92-e766-42eb-adbc-b6d17a65e8ea/6e4545c6-9e5c-4e6b-94f2-451b2f16f4ae"
-					(reference "R17")
-					(unit 1)
-				)
-				(path "/2ecddb92-e766-42eb-adbc-b6d17a65e8ea/92ea14e4-7796-41b2-9af7-4cb5ffd88b52"
-					(reference "R15")
-					(unit 1)
-				)
-				(path "/2ecddb92-e766-42eb-adbc-b6d17a65e8ea/d66c3d32-3008-485f-b8d3-7e1a6a0b22a4"
-					(reference "R32")
-					(unit 1)
-				)
-			)
-		)
-	)
-	(symbol
-		(lib_id "Device:R")
 		(at 130.81 82.55 270)
 		(unit 1)
@@
 					(unit 1)
 				)
-			)
-		)
-	)
-	(symbol
-		(lib_id "power:+3.3V")
-		(at 123.19 142.24 90)
-		(unit 1)
-		(exclude_from_sim no)
-		(in_bom yes)
-		(on_board yes)
-		(dnp no)
-		(property "Reference" "#PWR054"
-			(at 127 142.24 0)
-			(effects
-				(font
-					(size 1.27 1.27)
-				)
-				(hide yes)
-			)
-		)
-		(property "Value" "+3V3"
-			(at 119.38 142.2399 90)
-			(effects
-				(font
-					(size 1.27 1.27)
-				)
-				(justify left)
-			)
-		)
-		(property "Footprint" ""
-			(at 123.19 142.24 0)
-			(effects
-				(font
-					(size 1.27 1.27)
-				)
-				(hide yes)
-			)
-		)
-		(property "Datasheet" ""
-			(at 123.19 142.24 0)
-			(effects
-				(font
-					(size 1.27 1.27)
-				)
-				(hide yes)
-			)
-		)
-		(property "Description" "Power symbol creates a global label with name \"+3.3V\""
-			(at 123.19 142.24 0)
-			(effects
-				(font
-					(size 1.27 1.27)
-				)
-				(hide yes)
-			)
-		)
-		(pin "1"
-		)
-		(instances
-			(project "OZYS_V3_Final"
-				(path "/2ecddb92-e766-42eb-adbc-b6d17a65e8ea/55853f5b-0992-495b-b96a-8743589b5403"
-					(reference "#PWR054")
-					(unit 1)
-				)
-				(path "/2ecddb92-e766-42eb-adbc-b6d17a65e8ea/6e4545c6-9e5c-4e6b-94f2-451b2f16f4ae"
-					(reference "#PWR051")
-					(unit 1)
-				)
-				(path "/2ecddb92-e766-42eb-adbc-b6d17a65e8ea/92ea14e4-7796-41b2-9af7-4cb5ffd88b52"
-					(reference "#PWR049")
-					(unit 1)
-				)
-				(path "/2ecddb92-e766-42eb-adbc-b6d17a65e8ea/d66c3d32-3008-485f-b8d3-7e1a6a0b22a4"
-					(reference "#PWR070")
-					(unit 1)
-				)

Commit message: Pours fixed, no Graphics
Made sure all pours conform to 8mils clearance and width, with Solid connections.
Parts:
- renumbered R15 to R26
Changed lines of the file:
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@@
 		(dnp no)
 		(fields_autoplaced yes)
-		(property "Reference" "R15"
+		(property "Reference" "R26"
 			(at 167.64 135.89 90)
 			(effects
