File: epsilon_r2/epsilon_r2.kicad_pcb (KiCad board)
At the start: 2 copper layers, 17 x 12 mm, 18 parts, among them J1 SGP+, J2 SGS+, J3 SGP-, J4 SGS-, J5 AudioJack4, U2 DS28E07P+T, U3 TCA9416DDFR, U4 ADA4940-1ACPZ-R7

Commit message: epsilon_r2
Parts:
- C5, C6, C7, D1: moved to B.Cu
- moved R6 3.78 mm to (144.5, 85.3), turned to -90 degrees
- moved R5 3.35 mm to (146.2, 85.3), turned to -90 degrees
- moved C6 3.14 mm to (149.9, 86.0), turned to 90 degrees
- moved C5 3.13 mm to (149.0, 86.0), turned to -90 degrees
- moved C7 3.09 mm to (148.0, 86.0), turned to -90 degrees
- moved D1 1.49 mm to (149.3, 80.1), turned to 0 degrees
- moved U4 0.63 mm to (148.6, 86.0)
- moved U2 0.43 mm to (141.6, 82.0)
Routing:
- net GND: track 51.3 -> 35.0 mm, vias 5 -> 4
- net Net-(U4-+FB): track 3.12 -> 12.1 mm
- net Net-(U4-+IN): track 12.3 -> 17.5 mm
- net Net-(U4-–FB): track 3.26 -> 8.16 mm
- net Net-(D1-K): track 24.8 -> 21.0 mm, vias 5 -> 4
- net Net-(U4--OUT): track 12.3 -> 9.86 mm
- net Net-(U4--IN): track 18.2 -> 20.4 mm
- net 3V3A_SW: track 38.1 -> 36.3 mm, vias 3 -> 4
- net Net-(U4-+OUT): track 6.66 -> 5.40 mm, vias 1 -> 0
- net Net-(U4-VOCM): track 2.20 -> 2.26 mm, vias 0 -> 1
Other:
- board text added: "r2"
